File: Teensy base beta/schematic_base_board.sch (EAGLE design)
At the start: 25 parts, among them U1 SN754410NE, X4 22-23-2051, X5 22-23-2051

Commit message: working on design
Parts:
- removed V1: 7486N, 74ttl-din:7486N
- added IC1: 7486N, 74xx-us:7486N
- D1: value (none) -> 1N4004; device diode:DIODE-C2673 -> diode:1N4004
Connections:
- removed net N$11: _1._D7
- removed net N$12: _1._C6
- removed net N$13: _1._C7
- removed net N$24: _1._B0
- removed net N$25: _1._B1
- removed net N$26: _1._B2
- removed net N$27: _1._B3
- removed net N$28: _1._B4
- removed net N$3: U1.1,2EN
- removed net N$31: U1.3,4EN
- removed net N$32: U1.1A
- removed net N$33: U1.2A
- removed net N$34: U1.3A
- removed net N$35: U1.4A
- removed net N$4: _1._D0
- removed net N$5: _1._D1
- new net EN_A_L: U1.1A, _1._B1
- new net EN_A_R: U1.3A, _1._B2
- new net EN_B_L: U1.2A, _1._B0
- new net EN_B_R: U1.4A, _1._B3
- new net PWM_L: U1.1,2EN, _1._C6
- new net PWM_R: U1.3,4EN, _1._C7
- net CHA_ENC_L: now also IC1A.I0; no longer V1/1.A
- net CHA_ENC_R: now also IC1B.I0; no longer V1/2.A
- net CHB_ENC_L: now also IC1A.I1, _1._D7; no longer V1/1.B
- net CHB_ENC_R: now also IC1B.I1, _1._B4; no longer V1/2.B
- net GND: now also IC1C.I0, IC1C.I1, IC1D.I0, IC1D.I1, U1.GND_3; no longer V1/3.A, V1/3.B, V1/4.A, V1/4.B
- net INT_ENC_LEFT: now also IC1A.O, _1._D0; no longer V1/1.Y
- net INT_ENC_RIGHT: now also IC1B.O, _1._D1; no longer V1/2.Y
- net N$16: now also JP5.3
- net N$17: now also JP4.3
- net N$18: now also JP3.3
- net N$19: now also JP2.3
- net N$20: now also JP1.3
- net N$30: now also JP6.3
